Commit message: Changed constant

File: post_description/urdf/xtion.urdf.xacro (robot description, xacro)
@@ -72,5 +72,5 @@
         <parent link="xtion_proto_link"/>
         <child link="xtion_camera_link"/>
-        <origin xyz="0 0 0.07" rpy="0 0 3.1415"/>
+        <origin xyz="0 0 0.07" rpy="0 0 0"/>
         <axis xyz="0 0 1"/>
     </joint>

Commit message: Changed axis of xtion tilt

File: post_description/urdf/xtion.urdf.xacro (robot description, xacro)
@@ -59,5 +59,5 @@
         <parent link="xtion_inter_link"/>
         <child link="xtion_proto_link"/>
-        <axis xyz=" 1 0 0"/>
+        <axis xyz=" -1 0 0"/>
         <limit effort="1.0" velocity="1.0" lower="-3.1415" upper="3.1415"/>
     </joint>
