Commit message: New stuff

File: post_description/urdf/post.urdf.xacro (robot description, xacro)
@@ -33,5 +33,5 @@
         <axis xyz="0 0 0"/>
     </joint>
-    <joint name="spindar_joint" type="revolute">
+    <joint name="lidar_rad" type="revolute">
         <parent link="post_base"/>
         <child link="spindar_base"/>

File: post_description/urdf/xtion.urdf.xacro (robot description, xacro)
@@ -72,5 +72,5 @@
         <parent link="xtion_proto_link"/>
         <child link="xtion_camera_link"/>
-        <origin xyz="0 0 0.07" rpy="0 0 0"/>
+        <origin xyz="0 0 0.07" rpy="0 0 3.1415"/>
         <axis xyz="0 0 1"/>
     </joint>
@@ -87,4 +87,17 @@
             </geometry>
         </visual>
+    </link>
+    <joint name="xtion_etc1" type="fixed">
+        <parent link="xtion_camera_link"/>
+        <child link="camera_depth_optical_frame"/>
+        <origin xyz="0 0 0.0" rpy="1.5707 3.1415 0"/>
+        <axis xyz="0 0 1"/>
+    </joint>
+    <link name="camera_depth_optical_frame">
+      <inertial>
+        <origin xyz="0 0 0" rpy="0 0 0"/>
+        <mass value="0.01"/>
+        <inertia ixx="0.01"  ixy="0"  ixz="0" iyy="0.01" iyz="0" izz="0.01" />
+      </inertial>
     </link>
 <!--

Commit message: Got simulation and new nodes working

File: post_description/urdf/post.urdf.xacro (robot description, xacro)
@@ -1,4 +1,34 @@
 <?xml version="1.0"?>
 <robot xmlns:xacro="http://www.ros.org/wiki/xacro" name="post">
+    <transmission name="lidar_trans">
+      <type>transmission_interface/SimpleTransmission</type>
+      <joint name="lidar_rad">
+        <hardwareInterface>EffortJointInterface</hardwareInterface>
+      </joint>
+      <actuator name="lidar_motor">
+        <hardwareInterface>EffortJointInterface</hardwareInterface>
+        <mechanicalReduction>1</mechanicalReduction>
+      </actuator>
+    </transmission>
+    <transmission name="pan_trans">
+      <type>transmission_interface/SimpleTransmission</type>
+      <joint name="xtion_pan">
+        <hardwareInterface>EffortJointInterface</hardwareInterface>
+      </joint>
+      <actuator name="pan_motor">
+        <hardwareInterface>EffortJointInterface</hardwareInterface>
+        <mechanicalReduction>1</mechanicalReduction>
+      </actuator>
+    </transmission>
+    <transmission name="tilt_trans">
+      <type>transmission_interface/SimpleTransmission</type>
+      <joint name="xtion_tilt">
+        <hardwareInterface>EffortJointInterface</hardwareInterface>
+      </joint>
+      <actuator name="tilt_motor">
+        <hardwareInterface>EffortJointInterface</hardwareInterface>
+        <mechanicalReduction>1</mechanicalReduction>
+      </actuator>
+    </transmission>
     <xacro:include filename="$(find post_description)/urdf/xtion.urdf.xacro"/>
     <link name="post_base">
@@ -38,5 +68,5 @@
         <origin xyz="0 0 0.435" rpy="0 0 0"/>
         <axis xyz="1 0 0"/>
-        <limit effort="1.0" velocity="1.0" lower="-3.1415" upper="3.1415"/>
+        <limit effort="10.0" velocity="1.0" lower="-3.1415" upper="3.1415"/>
     </joint>
     <link name="spindar_base">
@@ -60,4 +90,5 @@
             </geometry>
       </visual>
+      <!--
       <collision>
             <origin xyz="0 0 0" rpy="0 0 0"/>
@@ -66,9 +97,72 @@
             </geometry>
       </collision>
+  -->
     </link>
     <gazebo>
         <plugin name="gazebo_ros_control" filename="libgazebo_ros_control.so">
-        <robotNamespace>/centaur</robotNamespace>
+        <robotNamespace>/post</robotNamespace>
         </plugin>
     </gazebo>
+    <gazebo reference="camera_depth_optical_frame">
+      <sensor name="xtion" type="depth">
+          <plugin name="camera_controller" filename="libgazebo_ros_openni_kinect.so">
+            <baseline>0.2</baseline>
+            <alwaysOn>true</alwaysOn>
+            <updateRate>1.0</updateRate>
+            <cameraName>camera_ir</cameraName>
+            <imageTopicName>/camera/depth/image_raw</imageTopicName>
+            <cameraInfoTopicName>/camera/depth/camera_info</cameraInfoTopicName>
+            <depthImageTopicName>/camera/depth/image_raw</depthImageTopicName>
+            <depthImageInfoTopicName>/camera/depth/camera_info</depthImageInfoTopicName>
+            <pointCloudTopicName>/camera/depth/points</pointCloudTopicName>
+            <frameName>camera_depth_optical_frame_virtual</frameName>
+            <pointCloudCutoff>0.5</pointCloudCutoff>
+            <distortionK1>0.00000001</distortionK1>
+            <distortionK2>0.00000001</distortionK2>
+            <distortionK3>0.00000001</distortionK3>
+            <distortionT1>0.00000001</distortionT1>
+            <distortionT2>0.00000001</distortionT2>
+            <CxPrime>0</CxPrime>
+            <Cx>0</Cx>
+            <Cy>0</Cy>
+            <focalLength>0</focalLength>
+            <hackBaseline>0</hackBaseline>
+          </plugin>
+      </sensor>
+    </gazebo>
+    <gazebo reference="laser">
+    <sensor type="ray" name="head_hokuyo_sensor">
+      <pose>0 0 0 0 0 0</pose>
+      <visualize>true</visualize>
+      <update_rate>10</update_rate>
+      <ray>
+        <scan>
+          <horizontal>
+            <samples>720</samples>
+            <resolution>1</resolution>
+            <min_angle>-1.570796</min_angle>
+            <max_angle>1.570796</max_angle>
+          </horizontal>
+        </scan>
+        <range>
+          <min>0.10</min>
+          <max>10.0</max>
+          <resolution>0.01</resolution>
+        </range>
+        <noise>
+          <type>gaussian</type>
+          <!-- Noise parameters based on published spec for Hokuyo laser
+               achieving "+-30mm" accuracy at range < 10m.  A mean of 0.0m and
+               stddev of 0.01m will put 99.7% of samples within 0.03m of the true
+               reading. -->
+          <mean>0.0</mean>
+          <stddev>0.01</stddev>
+        </noise>
+      </ray>
+      <plugin name="gazebo_ros_head_hokuyo_controller" filename="libgazebo_ros_laser.so">
+        <topicName>/laser</topicName>
+        <frameName>laser</frameName>
+      </plugin>
+    </sensor>
+  </gazebo>
 </robot>

File: post_description/urdf/xtion.urdf.xacro (robot description, xacro)
@@ -2,24 +2,4 @@
 <robot xmlns:xacro="http://www.ros.org/wiki/xacro">
   <xacro:parameter name="pi" value="3.1415"/>
-    <transmission name="xtion_pan_trans">
-      <type>transmission_interface/SimpleTransmission</type>
-      <joint name="xtion_pan">
-        <hardwareInterface>PositionJointInterface</hardwareInterface>
-      </joint>
-      <actuator name="xtion_pan_motor">
-        <hardwareInterface>PositionJointInterface</hardwareInterface>
-        <mechanicalReduction>1</mechanicalReduction>
-      </actuator>
-    </transmission>
-    <transmission name="xtion_tilt_trans">
-      <type>transmission_interface/SimpleTransmission</type>
-      <joint name="xtion_tilt">
-        <hardwareInterface>PositionJointInterface</hardwareInterface>
-      </joint>
-      <actuator name="xtion_tilt_motor">
-        <hardwareInterface>PositionJointInterface</hardwareInterface>
-        <mechanicalReduction>1</mechanicalReduction>
-      </actuator>
-    </transmission>
     <link name="xtion_base">
       <inertial>
@@ -40,5 +20,5 @@
         <origin xyz="0 0 0.075" rpy="0 0 0"/>
         <axis xyz="0 0 1"/>
-        <limit effort="1.0" velocity="1.0" lower="-3.1415" upper="3.1415"/>
+        <limit effort="100.0" velocity="1.0" lower="-3.1415" upper="3.1415"/>
     </joint>
     <link name="xtion_inter_link">
@@ -60,5 +40,5 @@
         <child link="xtion_proto_link"/>
         <axis xyz=" -1 0 0"/>
-        <limit effort="1.0" velocity="1.0" lower="-3.1415" upper="3.1415"/>
+        <limit effort="100.0" velocity="1.0" lower="-1.5707" upper="1.5707"/>
     </joint>
     <link name="xtion_proto_link">
@@ -90,6 +70,13 @@
     <joint name="xtion_etc1" type="fixed">
         <parent link="xtion_camera_link"/>
+        <child link="camera_frame_inter_link"/>
+        <origin xyz="0 0 0.0" rpy="0 0 0"/>
+        <axis xyz="0 0 1"/>
+    </joint>
+    <link name="camera_frame_inter_link"/>
+    <joint name="xtion_etc2" type="fixed">
+        <parent link="camera_frame_inter_link"/>
         <child link="camera_depth_optical_frame"/>
-        <origin xyz="0 0 0.0" rpy="1.5707 3.1415 0"/>
+        <origin xyz="0 0 0.0" rpy="0 0 -1.5707"/>
         <axis xyz="0 0 1"/>
     </joint>
@@ -101,4 +88,13 @@
       </inertial>
     </link>
+    <joint name="camera_optical_joint" type="fixed">
+    <!-- these values have to be these values otherwise the gazebo camera
+        image won't be aligned properly with the frame it is supposedly
+        originating from -->
+    <origin xyz="0 0 0" rpy="-1.5707 0 -1.5707"/>
+    <parent link="camera_depth_optical_frame"/>
+    <child link="camera_depth_optical_frame_virtual"/>
+  </joint>
+    <link name="camera_depth_optical_frame_virtual"/>
 <!--
     <gazebo reference="xtion_camera_link">

Commit message: Added new stuff and functionality

File: post_description/urdf/post.urdf.xacro (robot description, xacro)
@@ -72,4 +72,13 @@
     <link name="spindar_base">
     </link>
+    <joint name="lidar_base_joint" type="fixed">
+        <parent link="post_base"/>
+        <child link="lidar_base"/>
+        <origin xyz="0 0 0.435" rpy="0 0 0"/>
+        <axis xyz="1 0 0"/>
+        <limit effort="10.0" velocity="1.0" lower="-3.1415" upper="3.1415"/>
+    </joint>
+     <link name="lidar_base">
+     </link>
     <joint name="spindar_pos" type="fixed">
         <parent link="spindar_base"/>
